Commit message: Fixed issues

File: my_rb1_description/urdf/my_rb1_robot.xacro (robot description, xacro)
@@ -12,4 +12,26 @@
     <color rgba="0 0 1 0.5"/>
   </material>
+  <!-- Dummy link for KDL Warning correction-->
+  <link name="base_footprint">
+    <link name="base_footprint">
+    <inertial>
+        <origin xyz="0 0 0" rpy="0 0 0"/>
+        <mass value="0.001"/>
+        <inertia ixx="0.0001" ixy="0" ixz="0" iyy="0.0001" iyz="0" izz="0.0001"/>
+    </inertial>
+    <visual>
+        <origin xyz="0 0 0" rpy="0 0 0"/>
+        <geometry>
+        <box size="0.01 0.01 0.01"/>
+        </geometry>
+        <material name="grey"/>
+    </visual>
+    </link>
+  </link>
+  <joint name="chassis_joint" type="fixed">
+    <origin xyz="0 0 0" rpy="0 0 0"/>
+    <parent link="base_footprint"/>
+    <child link="base_link"/>
+  </joint>
   <!-- Base link -->
     <gazebo reference="base_link">
@@ -32,7 +54,7 @@
     </visual>
     <collision>
-      <origin xyz="0 0 0" rpy="0 0 0"/>
-      <geometry>
-        <cylinder radius="0.25" length="0.3"/>
+      <origin xyz="0 0 0.5" rpy="0 0 0"/>
+      <geometry>
+        <cylinder radius="0.25" length="0.1"/>
       </geometry>
     </collision>
@@ -42,5 +64,5 @@
     <parent link="base_link"/>
     <child link="left_wheel"/>
-    <origin xyz="0.0 -0.2 -0.15" rpy="0 0 0"/>
+    <origin xyz="0.0 0.2 -0.15" rpy="0 0 0"/>
     <axis xyz="0 1 0"/>
     <limit effort="10000" velocity="1000" />
@@ -54,17 +76,20 @@
     </inertial>
     <collision>
-        <origin rpy="0 0 0" xyz="0 0 0" />
-        <geometry>
-            <cylinder length="0.05" radius="0.025"/>
-        </geometry>
-    </collision>
-    <visual>
-      <origin xyz="0 0 0" rpy="0 0 0"/>
-      <geometry>
-        <cylinder radius="0.025" length="0.05"/>
+        <origin rpy="1.5708 0 0" xyz="0 0 0" />
+        <geometry>
+            <cylinder length="0.01" radius="0.025"/>
+        </geometry>
+    </collision>
+    <visual>
+      <origin xyz="0 0 0" rpy="1.5708 0 0"/>
+      <geometry>
+        <cylinder radius="0.025" length="0.01"/>
       </geometry>
       <material name="black"/>
     </visual>
   </link>
+    <gazebo reference="left_wheel">
+        <material>Gazebo/Red</material>
+    </gazebo>
 <!--Wheel Right-->
   <joint name="right_wheel_joint" type="continuous">
@@ -83,24 +108,52 @@
     </inertial>
     <collision>
-        <origin rpy="0 0 0" xyz="0 0 0" />
-        <geometry>
-            <cylinder length="0.05" radius="0.025"/>
-        </geometry>
-    </collision>
-    <visual>
-      <origin xyz="0 0 0" rpy="0 0 0"/>
-      <geometry>
-        <cylinder radius="0.025" length="0.05"/>
+        <origin rpy="1.5708 0 0" xyz="0 0 0" />
+        <geometry>
+            <cylinder length="0.01" radius="0.025"/>
+        </geometry>
+    </collision>
+    <visual>
+      <origin xyz="0 0 0" rpy="1.5708 0 0"/>
+      <geometry>
+        <cylinder radius="0.025" length="0.01"/>
       </geometry>
       <material name="black"/>
     </visual>
   </link>
+    <gazebo reference="right_wheel">
+        <material>Gazebo/Red</material>
+    </gazebo>
   <!-- caster wheel -->
   <joint name="front_caster_joint" type="fixed">
     <parent link="base_link"/>
     <child link="front_caster"/>
+    <origin xyz="0.1 0 -0.15" rpy="0 0 0"/>
+    <joint_properties friction="0.0" />
+  </joint>
+  <link name="front_caster">
+    <visual>
+      <origin xyz="0 0 0" rpy="0 0 0"/>
+      <geometry>
+        <sphere radius="0.0125"/>
+      </geometry>
+      <material name="grey"/>
+    </visual>
+    <collision>
+        <origin rpy="0 0 0" xyz="0 0 0" />
+        <geometry>
+            <sphere radius="0.0125"/>
+        </geometry>
+    </collision>
+  </link>
+    <gazebo reference="front_caster">
+        <material>Gazebo/White</material>
+    </gazebo>
+  <joint name="back_caster_joint" type="fixed">
+    <parent link="base_link"/>
+    <child link="back_caster"/>
     <origin xyz="-0.1 0 -0.15" rpy="0 0 0"/>
-  </joint>
-  <link name="front_caster">
+    <joint_properties friction="0.0" />
+  </joint>
+  <link name="back_caster">
     <visual>
       <origin xyz="0 0 0" rpy="0 0 0"/>
@@ -110,19 +163,14 @@
       <material name="grey"/>
     </visual>
-  </link>
-  <joint name="back_caster_joint" type="fixed">
-    <parent link="base_link"/>
-    <child link="back_caster"/>
-    <origin xyz="0.1 0 -0.15" rpy="0 0 0"/>
-  </joint>
-  <link name="back_caster">
-    <visual>
-      <origin xyz="0 0 0" rpy="0 0 0"/>
-      <geometry>
-        <sphere radius="0.0125"/>
-      </geometry>
-      <material name="grey"/>
-    </visual>
-  </link>
+    <collision>
+        <origin rpy="0 0 0" xyz="0 0 0" />
+        <geometry>
+            <sphere radius="0.0125"/>
+        </geometry>
+    </collision>
+  </link>
+    <gazebo reference="back_caster">
+        <material>Gazebo/White</material>
+    </gazebo>
     <gazebo>
         <plugin filename="libgazebo_ros_diff_drive.so" name="differential_drive_controller">

Commit message: Corrected friction issue of castor wheels

File: my_rb1_description/urdf/my_rb1_robot.xacro (robot description, xacro)
@@ -1,5 +1,4 @@
-<?xml version="1.0"?>
-<robot name="robot" xmlns:xacro="http://www.ros.org/wiki/xacro">
-  <!-- <xacro:include filename="$(find robot_description)/urdf/robot.gazebo" /> -->
+<?xml version="1.0" ?>
+<robot name="robot">
 <!-- Material Definitions -->
   <material name="black">
@@ -14,10 +13,4 @@
   <!-- Dummy link for KDL Warning correction-->
   <link name="base_footprint">
-    <link name="base_footprint">
-    <inertial>
-        <origin xyz="0 0 0" rpy="0 0 0"/>
-        <mass value="0.001"/>
-        <inertia ixx="0.0001" ixy="0" ixz="0" iyy="0.0001" iyz="0" izz="0.0001"/>
-    </inertial>
     <visual>
         <origin xyz="0 0 0" rpy="0 0 0"/>
@@ -27,5 +20,4 @@
         <material name="grey"/>
     </visual>
-    </link>
   </link>
   <joint name="chassis_joint" type="fixed">
@@ -66,6 +58,6 @@
     <origin xyz="0.0 0.2 -0.15" rpy="0 0 0"/>
     <axis xyz="0 1 0"/>
-    <limit effort="10000" velocity="1000" />
-    <joint_properties damping="1.0" friction="1.0" />
+    <limit effort="100" velocity="100" />
+    <joint_properties friction="1.0" />
   </joint>
   <link name="left_wheel">
@@ -76,7 +68,7 @@
     </inertial>
     <collision>
-        <origin rpy="1.5708 0 0" xyz="0 0 0" />
-        <geometry>
-            <cylinder length="0.01" radius="0.025"/>
+        <origin rpy="1.57079632679 0 0" xyz="0 0 0" />
+        <geometry>
+            <cylinder length="0.04" radius="0.025"/>
         </geometry>
     </collision>
@@ -84,5 +76,5 @@
       <origin xyz="0 0 0" rpy="1.5708 0 0"/>
       <geometry>
-        <cylinder radius="0.025" length="0.01"/>
+        <cylinder radius="0.025" length="0.04"/>
       </geometry>
       <material name="black"/>
@@ -98,6 +90,6 @@
     <origin xyz="0.0 -0.2 -0.15" rpy="0 0 0"/>
     <axis xyz="0 1 0"/>
-    <limit effort="10000" velocity="1000" />
-    <joint_properties damping="1.0" friction="1.0" />
+    <limit effort="100" velocity="100" />
+    <joint_properties friction="1.0" />
   </joint>
   <link name="right_wheel">
@@ -108,7 +100,7 @@
     </inertial>
     <collision>
-        <origin rpy="1.5708 0 0" xyz="0 0 0" />
-        <geometry>
-            <cylinder length="0.01" radius="0.025"/>
+        <origin rpy="1.57079632679 0 0" xyz="0 0 0" />
+        <geometry>
+            <cylinder length="0.04" radius="0.025"/>
         </geometry>
     </collision>
@@ -116,5 +108,5 @@
       <origin xyz="0 0 0" rpy="1.5708 0 0"/>
       <geometry>
-        <cylinder radius="0.025" length="0.01"/>
+        <cylinder radius="0.025" length="0.04"/>
       </geometry>
       <material name="black"/>
@@ -124,53 +116,90 @@
         <material>Gazebo/Red</material>
     </gazebo>
+  <gazebo reference="right_wheel">
+    <material>Gazebo/Red</material>
+    <surface>
+        <friction>
+        <ode>
+            <mu>1.5</mu>
+            <mu2>1.5</mu2>
+        </ode>
+        </friction>
+    </surface>
+  </gazebo>
+  <gazebo reference="left_wheel">
+    <material>Gazebo/Red</material>
+    <surface>
+        <friction>
+        <ode>
+            <mu>1.5</mu>
+            <mu2>1.5</mu2>
+        </ode>
+        </friction>
+    </surface>
+  </gazebo>
   <!-- caster wheel -->
-  <joint name="front_caster_joint" type="fixed">
+<link name="front_castor">
+    <inertial>
+        <mass value="0.1" />
+        <inertia ixx="0.0001" iyy="0.0001" izz="0.0001" ixy="0.0" ixz="0.0" iyz="0.0"/>
+    </inertial>
+    <visual>
+        <origin xyz="0 0 0" rpy="0 0 0"/>
+        <geometry>
+            <sphere radius="0.025"/>
+        </geometry>
+        <material name="black"/>
+    </visual>
+    <collision>
+        <origin xyz="0 0 0" rpy="0 0 0"/>
+        <geometry>
+            <sphere radius="0.025"/>
+        </geometry>
+    </collision>
+</link>
+<!-- Front caster wheel joint -->
+<joint name="front_castor_joint" type="fixed">
+    <origin xyz="-0.1 0.0 -0.15" rpy="0 0 0"/>
     <parent link="base_link"/>
-    <child link="front_caster"/>
-    <origin xyz="0.1 0 -0.15" rpy="0 0 0"/>
-    <joint_properties friction="0.0" />
-  </joint>
-  <link name="front_caster">
-    <visual>
-      <origin xyz="0 0 0" rpy="0 0 0"/>
-      <geometry>
-        <sphere radius="0.025"/>
-      </geometry>
-      <material name="grey"/>
-    </visual>
-    <collision>
-        <origin rpy="0 0 0" xyz="0 0 0" />
+    <child link="front_castor"/>
+</joint>
+<!-- Gazebo plugin for front caster wheel to set friction to zero -->
+<gazebo reference="front_castor">
+    <material>Gazebo/White</material>
+    <mu1>0.0</mu1> <!-- Friction parameter -->
+    <mu2>0.0</mu2> <!-- Friction parameter -->
+</gazebo>
+<!-- Back caster wheel link -->
+<link name="back_castor">
+    <inertial>
+        <mass value="0.1" />
+        <inertia ixx="0.0001" iyy="0.0001" izz="0.0001" ixy="0.0" ixz="0.0" iyz="0.0"/>
+    </inertial>
+    <visual>
+        <origin xyz="0 0 0" rpy="0 0 0"/>
         <geometry>
             <sphere radius="0.025"/>
         </geometry>
-    </collision>
-  </link>
-    <gazebo reference="front_caster">
-        <material>Gazebo/White</material>
-    </gazebo>
-  <joint name="back_caster_joint" type="fixed">
+        <material name="black"/>
+    </visual>
+    <collision>
+        <origin xyz="0 0 0" rpy="0 0 0"/>
+        <geometry>
+            <sphere radius="0.025"/>
+        </geometry>
+    </collision>
+</link>
+<!-- Back caster wheel joint -->
+<joint name="back_castor_joint" type="fixed">
+    <origin xyz="0.1 0.0 -0.15" rpy="0 0 0"/>
     <parent link="base_link"/>
-    <child link="back_caster"/>
-    <origin xyz="-0.1 0 -0.15" rpy="0 0 0"/>
-    <joint_properties friction="0.0" />
-  </joint>
-  <link name="back_caster">
-    <visual>
-      <origin xyz="0 0 0" rpy="0 0 0"/>
-      <geometry>
-        <sphere radius="0.0025"/>
-      </geometry>
-      <material name="grey"/>
-    </visual>
-    <collision>
-        <origin rpy="0 0 0" xyz="0 0 0" />
-        <geometry>
-            <sphere radius="0.025"/>
-        </geometry>
-    </collision>
-  </link>
-    <gazebo reference="back_caster">
-        <material>Gazebo/White</material>
-    </gazebo>
+    <child link="back_castor"/>
+</joint>
+<!-- Gazebo plugin for back caster wheel to set friction to zero -->
+<gazebo reference="back_castor">
+    <material>Gazebo/White</material>
+    <mu1>0.0</mu1> <!-- Friction parameter -->
+    <mu2>0.0</mu2> <!-- Friction parameter -->
+</gazebo>
     <gazebo>
         <plugin filename="libgazebo_ros_diff_drive.so" name="differential_drive_controller">
