Commit message: Corrected the wheel positions and base_footprint visual

File: my_rb1_description/urdf/my_rb1_robot.urdf (robot description, URDF)
Before this commit: robot my_rb1_robot, 7 links, 6 joints
Links:
- removed link link_chassis
- added link base_footprint
Joints:
- joint back_caster_joint: origin xyz=0.1 0 -0.15 rpy=0 0 0 -> xyz=-0.1 0 -0.15 rpy=0 0 0
- joint chassis_joint: parent link_chassis -> base_footprint
- joint front_caster_joint: origin xyz=-0.1 0 -0.15 rpy=0 0 0 -> xyz=0.1 0 -0.15 rpy=0 0 0
- joint left_wheel_joint: origin xyz=0.0 -0.2 -0.15 rpy=0 0 0 -> xyz=0.0 0.2 -0.15 rpy=0 0 0
- joint right_wheel_joint: origin xyz=0.0 0.2 -0.15 rpy=0 0 0 -> xyz=0.0 -0.2 -0.15 rpy=0 0 0

Commit message: Corrected castor wheel position

File: my_rb1_description/urdf/my_rb1_robot.urdf (robot description, URDF)
Before this commit: robot my_rb1_robot, 7 links, 6 joints
Links:
- link back_caster: geometry collision sphere radius=0.025; visual sphere radius=0.025
- link base_link: geometry collision cylinder length=0.1 radius=0.25; visual cylinder length=0.3 radius=0.25
- link front_caster: geometry collision sphere radius=0.025; visual sphere radius=0.025
- link left_wheel: mass None -> 1; geometry collision cylinder length=0.02 radius=0.025; visual cylinder length=0.02 radius=0.025
- link link_laser_scan: mass None -> 0.5; geometry collision cylinder length=0.075 radius=0.05; visual cylinder length=0.075 radius=0.05
- link right_wheel: mass None -> 1; geometry collision cylinder length=0.02 radius=0.025; visual cylinder length=0.02 radius=0.025
Joints:
- removed joint laser_joint
- added joint joint_laser_scan_chassis: type fixed, parent base_link, child link_laser_scan, origin xyz=0.25 0 0.075 rpy=3.14159 0 0
- joint chassis_joint: origin xyz=0 0 0 rpy=0 0 0 -> xyz=0 0 0.15 rpy=0 0 0
- joint left_wheel_joint: limit effort=0 velocity=0 -> effort=10000 velocity=1000
- joint right_wheel_joint: limit effort=0 velocity=0 -> effort=10000 velocity=1000

File: my_rb1_description/urdf/my_rb1_robot.xacro (robot description, xacro)
@@ -30,5 +30,5 @@
   </link>
   <joint name="chassis_joint" type="fixed">
-    <origin xyz="0 0 0" rpy="0 0 0"/>
+    <origin xyz="0 0 0.15" rpy="0 0 0"/>
     <parent link="base_footprint"/>
     <child link="base_link"/>
@@ -135,5 +135,5 @@
       <origin xyz="0 0 0" rpy="0 0 0"/>
       <geometry>
-        <sphere radius="0.0125"/>
+        <sphere radius="0.025"/>
       </geometry>
       <material name="grey"/>
@@ -142,5 +142,5 @@
         <origin rpy="0 0 0" xyz="0 0 0" />
         <geometry>
-            <sphere radius="0.0125"/>
+            <sphere radius="0.025"/>
         </geometry>
     </collision>
@@ -159,5 +159,5 @@
       <origin xyz="0 0 0" rpy="0 0 0"/>
       <geometry>
-        <sphere radius="0.0125"/>
+        <sphere radius="0.0025"/>
       </geometry>
       <material name="grey"/>
@@ -166,5 +166,5 @@
         <origin rpy="0 0 0" xyz="0 0 0" />
         <geometry>
-            <sphere radius="0.0125"/>
+            <sphere radius="0.025"/>
         </geometry>
     </collision>

Commit message: Updated castor wheel properties

File: my_rb1_description/urdf/my_rb1_robot.urdf (robot description, URDF)
Before this commit: robot my_rb1_robot, 7 links, 6 joints
Links:
- removed link back_caster
- removed link front_caster
- added link back_castor, mass 0.1; collision sphere radius=0.025; visual sphere radius=0.025
- added link front_castor, mass 0.1; collision sphere radius=0.025; visual sphere radius=0.025
- link base_footprint: geometry collision cylinder length=0.001 radius=0.005; visual cylinder length=0.001 radius=0.005
- link base_link: geometry collision cylinder length=0.1 radius=0.25; visual cylinder length=0.3 radius=0.25
- link left_wheel: mass None -> 1; geometry collision cylinder length=0.04 radius=0.025; visual cylinder length=0.04 radius=0.025
- link link_laser_scan: mass None -> 0.5; geometry collision cylinder length=0.075 radius=0.05; visual cylinder length=0.075 radius=0.05
- link right_wheel: mass None -> 1; geometry collision cylinder length=0.04 radius=0.025; visual cylinder length=0.04 radius=0.025
Joints:
- removed joint back_caster_joint
- removed joint front_caster_joint
- removed joint laser_joint
- added joint back_castor_joint: type fixed, parent base_link, child back_castor, origin xyz=0.1 0.0 -0.15 rpy=0 0 0
- added joint front_castor_joint: type fixed, parent base_link, child front_castor, origin xyz=-0.1 0.0 -0.15 rpy=0 0 0
- added joint joint_laser_scan_chassis: type fixed, parent base_link, child link_laser_scan, origin xyz=0.25 0 0.075 rpy=3.14159 0 0
- joint chassis_joint: origin xyz=0 0 0 rpy=0 0 0 -> xyz=0 0 0.15 rpy=0 0 0
- joint left_wheel_joint: limit effort=0 velocity=0 -> effort=100 velocity=100
- joint right_wheel_joint: limit effort=0 velocity=0 -> effort=100 velocity=100

Commit message: Updated castor positions

File: my_rb1_description/urdf/my_rb1_robot.urdf (robot description, URDF)
Before this commit: robot robot, 7 links, 6 joints
Joints:
- joint back_castor_joint: origin xyz=0.1 0.0 -0.15 rpy=0 0 0 -> xyz=-0.1 0.0 -0.15 rpy=0 0 0
- joint front_castor_joint: origin xyz=-0.1 0.0 -0.15 rpy=0 0 0 -> xyz=0.1 0.0 -0.15 rpy=0 0 0
